Commit message: added lidar urdf, gazebo to be tested

File: src/robot_description/robot/robot.urdf.xacro (robot description, xacro)
@@ -5,4 +5,5 @@
     <xacro:include filename="$(find robot_description)/urdf/wheel_roller/wheel_roller.urdf.xacro"/>
     <xacro:include filename="$(find robot_description)/urdf/top/top.urdf.xacro"/>
+    <xacro:include filename="$(find robot_description)/urdf/lrf/lrf.urdf.xacro"/>
     <xacro:property name="chassis_radius" value="0.26"/>
     <xacro:property name="chassis_wheel_separation" value="0.018"/>
@@ -166,4 +167,8 @@
     </xacro:macro>
     <xacro:loop_rollers_wheel_back_out links_qty="7"/>
+    <!-- lrf sensor -->
+    <xacro:lrf_v0 parent="base_link">
+        <origin xyz="0 0 0.352" rpy="0 0 0"/>
+    </xacro:lrf_v0>
     <!-- ================= TRANSMISSIONS ================= -->
     <xacro:wheel_trans_v0 prefix="left"/>
@@ -187,3 +192,5 @@
     <xacro:wheel_gazebo_v0 prefix="front"/>
     <xacro:wheel_gazebo_v0 prefix="back"/>
+    <!-- lrf sensor -->
+    <xacro:lrf_gazebo_v0 min_rad = "-3.14" max_rad = "3.14" min_range = "0.1" max_range = "10"/>
 </robot>
